Commit message: Improve demo for latest Isaac ROS

File: isaac_ros/src/carter_description/urdf/carter.urdf (robot description, URDF)
Before this commit: robot carter, 8 links, 7 joints
Links:
- link rear_wheel_link: geometry collision sphere radius=.076; visual mesh filename=package://carter_description/urdf/meshes/caster_wheel.obj
